File: hillside48/hillside.kicad_sch (KiCad schematic)
At the start: 66 parts, among them J1 Haptic, J2 TRRS, J3 Bat_Pos, J4 Bat_GND, J5 Bat_Pos, J6 Bat_GND, K1 SW_Key, K10 SW_Key, K11 SW_Key, K12 SW_Key, K13 SW_Key, K14 SW_Key, K15 SW_Key, K16 SW_Key, K17 SW_Key, K18 SW_Key, K19 SW_Key, K2 SW_Key, K20 SW_Rotary, K21 SW_Key, K22 SW_Key, K23 SW_Key, K24 SW_Key, K3 SW_Key, K4 SW_Key, K5 SW_Key, K6 SW_Key, K7 SW_Key, K8 SW_Key, K9 SW_Key, SW1 Reset, SW2 SW_Power, U1 ProMicro_r

Commit message: footprint
Parts:
- removed H3: Logo, hillside:Hillside_Logo, symbol hillside:Logo
- added U2: XIAO-nRF52840-SMD, Seeed Studio XIAO Series Library:XIAO-nRF52840-SMD-2-sided, symbol Seeed_Studio_XIAO_Series:XIAO-nRF52840-SMD
Connections:
- net GND: now also U2.13 (GND), U2.18 (GND), U2.20 (GND)
- net LED: now also U2.7 (D6)
- net VCC: now also U2.12 (3V3_OUT)
- net col0: now also U2.1 (D0)
- net col1: now also U2.2 (D1)
- net col2: now also U2.3 (D2)
- net col3: now also U2.4 (D3)
- net col4: now also U2.5 (D4)
- net col5: now also U2.6 (D5)
- net raw: now also U2.19 (VBAT)
- net reset: now also U2.17 (EN)
- net row0: now also U2.8 (D7)
- net row1: now also U2.9 (D8)
- net row2: now also U2.10 (D9)
- net row3: now also U2.11 (D10)
- no-connect marks 5 -> 9
Other:
- moved on the sheet: J2, SW1, U1
